File: hat_v2.brd (EAGLE design)
At the start: 65 x 56.5 mm, 18 parts, among them IC1 4N35

Commit message: V2 board done
Parts:
- moved R5 194.9 mm to (54.9, 35.6), turned to 270 degrees
- moved IC1 166.9 mm to (33.0, 32.5), turned to 90 degrees
- moved J2 96.1 mm to (60.5, 38.1), turned to 270 degrees
- moved J1 82.9 mm to (60.5, 21.8), turned to 270 degrees
- moved C2 38.2 mm to (22.9, 32.5)
- moved C1 38.2 mm to (22.9, 41.7)
- moved VD2 33.2 mm to (44.7, 10.7), turned to 180 degrees
- moved D1 30.2 mm to (48.3, 27.4)
- moved ADS1115 21.8 mm to (32.5, 45.7), turned to 0 degrees
- moved GPS 15.2 mm to (3.81, 45.7)
- moved VD1 13.7 mm to (44.7, 18.8), turned to 180 degrees
- moved R3 10.4 mm to (51.8, 35.6)
- moved R4 10.1 mm to (48.5, 35.6)
- moved R1 9.76 mm to (45.0, 35.6)
- moved R2 9.45 mm to (41.7, 35.6)
Connections:
- net BAT-1: now also ADS1115.3; no longer ADS1115.4
- net BAT-2: now also ADS1115.4; no longer ADS1115.3
Routing:
- net 3.3V: track 0.00 -> 99.7 mm, vias 0 -> 1
- net SDA: track 0.00 -> 95.2 mm, vias 0 -> 2
- net SCL: track 0.00 -> 89.8 mm, vias 0 -> 2
- net GPIO5: track 0.00 -> 59.6 mm
- net BAT-2: track 0.00 -> 46.9 mm
- net BAT-2-INPUT: track 0.00 -> 37.3 mm
- net SHUNT-LOW-INPUT: track 0.00 -> 35.0 mm, vias 0 -> 1
- net BAT-1: track 0.00 -> 33.7 mm
- net SHUNT-HIGH-INPUT: track 0.00 -> 31.3 mm, vias 0 -> 1
- net GPIO18: track 0.00 -> 27.8 mm, vias 0 -> 1
- net BAT-1-INPUT: track 0.00 -> 24.9 mm
- net N$3: track 0.00 -> 20.8 mm
- net RXD: track 0.00 -> 19.7 mm
- net LINKED-INPUT: track 0.00 -> 13.6 mm
- net N$1: track 0.00 -> 11.2 mm
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
Commit message: Minor tweak to PCB
Parts:
- moved ADS1115 1.02 mm to (31.5, 45.7)
Routing:
- net SDA: track 95.2 -> 92.1 mm
- net SCL: track 89.8 -> 88.8 mm
- net 3.3V: track 99.7 -> 98.7 mm
- net BAT-2: track 46.9 -> 47.6 mm
Changed lines of the file:
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@@
 Design by:
 Andrew LeCody</text>
-<text x="52.832" y="43.942" size="0.762" layer="25" rot="R315">GND</text>
-<text x="55.372" y="43.942" size="0.762" layer="25" rot="R315">3.3v</text>
+<text x="51.816" y="43.942" size="0.762" layer="25" rot="R315">GND</text>
+<text x="54.356" y="43.942" size="0.762" layer="25" rot="R315">3.3v</text>
 <text x="29.21" y="5.588" size="0.762" layer="25" rot="R45">GND</text>
 <text x="26.67" y="5.588" size="0.762" layer="25" rot="R45">3.3v</text>
 <text x="13.97" y="5.588" size="0.762" layer="25" rot="R45">SDA</text>
 <text x="11.43" y="5.588" size="0.762" layer="25" rot="R45">SCL</text>
-<text x="50.292" y="43.942" size="0.762" layer="25" rot="R315">SCL</text>
-<text x="47.752" y="43.942" size="0.762" layer="25" rot="R315">SDA</text>
+<text x="49.276" y="43.942" size="0.762" layer="25" rot="R315">SCL</text>
+<text x="46.736" y="43.942" size="0.762" layer="25" rot="R315">SDA</text>
 </plain>
 <attributes>
@@
 <element name="R3" library="SparkFun-Passives" package="AXIAL-0.3" value="4k7" x="51.816" y="35.56" rot="R90"/>
 <element name="R4" library="SparkFun-Passives" package="AXIAL-0.3" value="1k" x="48.514" y="35.56" rot="R90"/>
-<element name="ADS1115" library="SparkFun-Connectors" package="1X10" value="" x="32.512" y="45.72">
-<attribute name="PROD_ID" value="CONN-11563" x="32.512" y="45.72" size="1.778" layer="27" display="off"/>
+<element name="ADS1115" library="SparkFun-Connectors" package="1X10" value="" x="31.496" y="45.72">
+<attribute name="PROD_ID" value="CONN-11563" x="31.496" y="45.72" size="1.778" layer="27" display="off"/>
 </element>
 <element name="ADXL345" library="SparkFun-Connectors" package="1X08" value="" x="29.21" y="3.81" rot="R180">
@@
 <contactref element="ADS1115" pad="7"/>
 <contactref element="ADXL345" pad="7"/>
-<wire x1="47.752" y1="45.72" x2="47.752" y2="44.196" width="0.4064" layer="1"/>
-<wire x1="47.752" y1="44.196" x2="47.244" y2="43.688" width="0.4064" layer="1"/>
-<wire x1="47.244" y1="43.688" x2="42.164" y2="43.688" width="0.4064" layer="1"/>
-<via x="42.164" y="43.688" extent="1-16" drill="0.6" diameter="0.4064" shape="square"/>
-<wire x1="42.164" y1="43.688" x2="30.988" y2="43.688" width="0.4064" layer="16"/>
-<via x="30.988" y="43.688" extent="1-16" drill="0.6" diameter="0.4064" shape="square"/>
-<wire x1="30.988" y1="43.688" x2="26.924" y2="47.752" width="0.4064" layer="1"/>
-<wire x1="26.924" y1="47.752" x2="14.388" y2="47.752" width="0.4064" layer="1"/>
+<wire x1="46.736" y1="45.72" x2="46.736" y2="44.196" width="0.4064" layer="1"/>
+<wire x1="46.736" y1="44.196" x2="46.228" y2="43.688" width="0.4064" layer="1"/>
+<wire x1="46.228" y1="43.688" x2="42.672" y2="43.688" width="0.4064" layer="1"/>
+<via x="42.672" y="43.688" extent="1-16" drill="0.6" diameter="0.4064" shape="square"/>
+<wire x1="42.672" y1="43.688" x2="28.956" y2="43.688" width="0.4064" layer="16"/>
+<via x="28.956" y="43.688" extent="1-16" drill="0.6" diameter="0.4064" shape="square"/>
+<wire x1="28.956" y1="43.688" x2="24.892" y2="47.752" width="0.4064" layer="1"/>
+<wire x1="24.892" y1="47.752" x2="14.388" y2="47.752" width="0.4064" layer="1"/>
 <wire x1="14.388" y1="47.752" x2="10.91" y2="51.23" width="0.4064" layer="1"/>
 <wire x1="13.97" y1="3.81" x2="13.97" y2="37.846" width="0.4064" layer="1"/>
 <wire x1="13.97" y1="37.846" x2="19.812" y2="43.688" width="0.4064" layer="1"/>
-<wire x1="19.812" y1="43.688" x2="30.988" y2="43.688" width="0.4064" layer="1"/>
+<wire x1="19.812" y1="43.688" x2="28.956" y2="43.688" width="0.4064" layer="1"/>
 </signal>
 <signal name="SCL">
@@
 <contactref element="ADS1115" pad="8"/>
 <contactref element="ADXL345" pad="8"/>
-<wire x1="50.292" y1="45.72" x2="50.292" y2="46.736" width="0.4064" layer="1"/>
-<wire x1="50.292" y1="46.736" x2="49.784" y2="47.244" width="0.4064" layer="1"/>
-<wire x1="49.784" y1="47.244" x2="44.704" y2="47.244" width="0.4064" layer="1"/>
+<wire x1="49.276" y1="45.72" x2="49.276" y2="46.736" width="0.4064" layer="1"/>
+<wire x1="49.276" y1="46.736" x2="48.768" y2="47.244" width="0.4064" layer="1"/>
+<wire x1="48.768" y1="47.244" x2="44.704" y2="47.244" width="0.4064" layer="1"/>
 <wire x1="44.704" y1="47.244" x2="43.18" y2="48.768" width="0.4064" layer="1"/>
-<wire x1="43.18" y1="48.768" x2="24.384" y2="48.768" width="0.4064" layer="1"/>
+<wire x1="43.18" y1="48.768" x2="23.876" y2="48.768" width="0.4064" layer="1"/>
 <wire x1="23.876" y1="48.768" x2="15.912" y2="48.768" width="0.4064" layer="1"/>
 <wire x1="15.912" y1="48.768" x2="13.45" y2="51.23" width="0.4064" layer="1"/>
@@
 <wire x1="20.32" y1="45.212" x2="23.876" y2="48.768" width="0.4064" layer="16"/>
 <via x="23.876" y="48.768" extent="1-16" drill="0.6" diameter="0.4064" shape="square"/>
-<wire x1="23.876" y1="48.768" x2="24.384" y2="48.768" width="0.4064" layer="1"/>
 </signal>
 <signal name="GPIO4">
@@
 <wire x1="59.436" y1="42.164" x2="59.944" y2="42.672" width="0.4064" layer="1"/>
 <wire x1="59.944" y1="42.672" x2="59.944" y2="47.752" width="0.4064" layer="1"/>
-<wire x1="59.944" y1="47.752" x2="58.928" y2="48.768" width="0.4064" layer="1"/>
-<wire x1="58.928" y1="48.768" x2="46.392" y2="48.768" width="0.4064" layer="1"/>
-<wire x1="46.392" y1="48.768" x2="43.93" y2="51.23" width="0.4064" layer="1"/>
+<wire x1="59.944" y1="47.752" x2="58.42" y2="49.276" width="0.4064" layer="1"/>
+<wire x1="58.42" y1="49.276" x2="45.884" y2="49.276" width="0.4064" layer="1"/>
+<wire x1="45.884" y1="49.276" x2="43.93" y2="51.23" width="0.4064" layer="1"/>
 </signal>
 <signal name="GPIO6">
@@
 <contactref element="ADXL345" pad="2"/>
 <contactref element="GPS" pad="2"/>
-<wire x1="55.372" y1="45.72" x2="55.372" y2="47.244" width="0.4064" layer="1"/>
-<wire x1="55.372" y1="47.244" x2="54.864" y2="47.752" width="0.4064" layer="1"/>
-<wire x1="54.864" y1="47.752" x2="45.72" y2="47.752" width="0.4064" layer="1"/>
-<wire x1="45.72" y1="47.752" x2="43.688" y2="49.784" width="0.4064" layer="1"/>
+<wire x1="54.356" y1="45.72" x2="54.356" y2="47.244" width="0.4064" layer="1"/>
+<wire x1="54.356" y1="47.244" x2="53.34" y2="48.26" width="0.4064" layer="1"/>
+<wire x1="53.34" y1="48.26" x2="45.212" y2="48.26" width="0.4064" layer="1"/>
+<wire x1="45.212" y1="48.26" x2="43.688" y2="49.784" width="0.4064" layer="1"/>
 <wire x1="43.688" y1="49.784" x2="30.136" y2="49.784" width="0.4064" layer="1"/>
 <wire x1="30.136" y1="49.784" x2="28.69" y2="51.23" width="0.4064" layer="1"/>
@@
 <wire x1="44.958" y1="39.37" x2="41.656" y2="39.37" width="0.4064" layer="1"/>
 <contactref element="ADS1115" pad="3"/>
-<wire x1="41.656" y1="39.37" x2="37.592" y2="43.434" width="0.4064" layer="1"/>
-<wire x1="37.592" y1="43.434" x2="37.592" y2="45.72" width="0.4064" layer="1"/>
+<wire x1="41.656" y1="39.37" x2="36.576" y2="44.45" width="0.4064" layer="1"/>
+<wire x1="36.576" y1="44.45" x2="36.576" y2="45.72" width="0.4064" layer="1"/>
 <wire x1="21.59" y1="41.656" x2="21.59" y2="40.386" width="0.4064" layer="1"/>
 <wire x1="21.59" y1="40.386" x2="23.368" y2="38.608" width="0.4064" layer="1"/>
@@
 <contactref element="ADS1115" pad="4"/>
 <wire x1="48.514" y1="39.37" x2="45.72" y2="42.164" width="0.4064" layer="1"/>
-<wire x1="45.72" y1="42.164" x2="41.656" y2="42.164" width="0.4064" layer="1"/>
-<wire x1="41.656" y1="42.164" x2="40.132" y2="43.688" width="0.4064" layer="1"/>
-<wire x1="40.132" y1="43.688" x2="40.132" y2="45.72" width="0.4064" layer="1"/>
+<wire x1="45.72" y1="42.164" x2="41.148" y2="42.164" width="0.4064" layer="1"/>
+<wire x1="41.148" y1="42.164" x2="39.116" y2="44.196" width="0.4064" layer="1"/>
+<wire x1="39.116" y1="44.196" x2="39.116" y2="45.72" width="0.4064" layer="1"/>
 <wire x1="21.59" y1="32.512" x2="21.59" y2="35.306" width="0.4064" layer="1"/>
 <wire x1="21.59" y1="35.306" x2="23.368" y2="37.084" width="0.4064" layer="1"/>
@@
 <wire x1="41.656" y1="36.576" x2="36.576" y2="41.656" width="0.4064" layer="16"/>
 <via x="36.576" y="41.656" extent="1-16" drill="0.6" diameter="0.4064" shape="square"/>
-<wire x1="36.576" y1="41.656" x2="35.052" y2="43.18" width="0.4064" layer="1"/>
-<wire x1="35.052" y1="43.18" x2="35.052" y2="45.72" width="0.4064" layer="1"/>
+<wire x1="36.576" y1="41.656" x2="34.036" y2="44.196" width="0.4064" layer="1"/>
+<wire x1="34.036" y1="44.196" x2="34.036" y2="45.72" width="0.4064" layer="1"/>
 </signal>
 <signal name="SHUNT-LOW-INPUT">
 <contactref element="J2" pad="2"/>
 <contactref element="ADS1115" pad="1"/>
-<wire x1="32.512" y1="45.72" x2="32.512" y2="42.672" width="0.4064" layer="1"/>
-<wire x1="32.512" y1="42.672" x2="33.528" y2="41.656" width="0.4064" layer="1"/>
+<wire x1="31.496" y1="45.72" x2="31.496" y2="43.688" width="0.4064" layer="1"/>
+<wire x1="31.496" y1="43.688" x2="33.528" y2="41.656" width="0.4064" layer="1"/>
 <via x="33.528" y="41.656" extent="1-16" drill="0.6" diameter="0.4064" shape="square"/>
 <wire x1="33.528" y1="41.656" x2="39.624" y2="35.56" width="0.4064" layer="16"/>

Commit message: Minor tweaks to v2
Parts:
- moved D1 7.40 mm to (41.1, 25.4)
- moved VD2 3.59 mm to (41.1, 10.2)
- moved VD1 3.56 mm to (41.1, 18.8)
- moved IC1 0.51 mm to (33.0, 32.0)
Routing:
- net BAT-1-INPUT: track 24.9 -> 31.3 mm
- net N$1: track 11.2 -> 15.7 mm
- net BAT-2-INPUT: track 37.3 -> 41.0 mm
Other:
- board text added: "Bat 1"
- board text added: "Bat 2"
- board text added: "Design By: Andrew LeCody"
- board text added: "Jeep Monitoring v2"
- board text added: "Linked"
- board text added: "Shunt High Shunt Low"
- board text removed: "Jeep Monitoring Design by: Andrew LeCody"
- board text removed: "Jeep Monitoring v1"
