File: hat_v2.sch (EAGLE design)
At the start: 18 parts, among them IC1 4N35

Commit message: V2 board done
Connections:
- net BAT-1: now also ADS1115.3; no longer ADS1115.4
- net BAT-2: now also ADS1115.4; no longer ADS1115.3
Changed lines of the file:
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@@
 </segment>
 <segment>
-<pinref part="ADS1115" gate="G$1" pin="4"/>
-<wire x1="17.78" y1="73.66" x2="22.86" y2="73.66" width="0.1524" layer="91"/>
-<label x="20.32" y="73.66" size="1.778" layer="95"/>
+<pinref part="ADS1115" gate="G$1" pin="3"/>
+<wire x1="17.78" y1="71.12" x2="22.86" y2="71.12" width="0.1524" layer="91"/>
+<label x="20.32" y="71.12" size="1.778" layer="95"/>
 </segment>
 </net>
@@
 </segment>
 <segment>
-<pinref part="ADS1115" gate="G$1" pin="3"/>
-<wire x1="17.78" y1="71.12" x2="22.86" y2="71.12" width="0.1524" layer="91"/>
-<label x="20.32" y="71.12" size="1.778" layer="95"/>
+<pinref part="ADS1115" gate="G$1" pin="4"/>
+<wire x1="17.78" y1="73.66" x2="22.86" y2="73.66" width="0.1524" layer="91"/>
+<label x="20.32" y="73.66" size="1.778" layer="95"/>
 </segment>
 </net>

Commit message: Minor tweaks to v2
Other:
- note added: "v2"
- note removed: "v1"
Changed lines of the file:
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@@
 <plain>
 <text x="149.86" y="7.62" size="2.54" layer="94">Andrew LeCody</text>
-<text x="241.3" y="7.62" size="2.54" layer="94">v1</text>
+<text x="241.3" y="7.62" size="2.54" layer="94">v2</text>
 </plain>
 <instances>
@@
 </sheet>
 </sheets>
+<errors>
+</errors>
 </schematic>
 </drawing>
